Commit message: 把抬脚和G1对齐

File: src/wbc_mjlab/CASBOT02_7dof/urdf/CASBOT02_ENCOS_22dof_shell_20251015.urdf (robot description, URDF)
Before this commit: robot CB02_URDF(ECS)130C, 32 links, 31 joints
Joints:
- joint leg_l1_joint: limit lower=-1.9199 upper=1.5708 effort=69.2 velocity=12.56 -> lower=-1.9199 upper=1.5708 effort=150 velocity=12.56
- joint leg_l2_joint: limit lower=-0.17453 upper=1.5708 effort=69.2 velocity=12.56 -> lower=-0.17453 upper=1.5708 effort=150 velocity=12.56
- joint leg_l3_joint: limit lower=-1.5708 upper=1.5708 effort=35.2 velocity=12.56 -> lower=-1.5708 upper=1.5708 effort=120 velocity=12.56
- joint leg_l4_joint: limit lower=0 upper=2.5307 effort=69.2 velocity=12.56 -> lower=0 upper=2.5307 effort=150 velocity=12.56
- joint leg_l5_joint: limit lower=-0.87266 upper=0.50614 effort=35.2 velocity=12.56 -> lower=-0.87266 upper=0.50614 effort=120 velocity=12.56
- joint leg_l6_joint: limit lower=-0.50614 upper=0.50614 effort=35.2 velocity=12.56 -> lower=-0.50614 upper=0.50614 effort=120 velocity=12.56
- joint leg_r1_joint: limit lower=-1.9199 upper=1.5708 effort=69.2 velocity=12.56 -> lower=-1.9199 upper=1.5708 effort=150 velocity=12.56
- joint leg_r2_joint: limit lower=-1.5708 upper=0.17453 effort=69.2 velocity=12.56 -> lower=-1.5708 upper=0.17453 effort=150 velocity=12.56
- joint leg_r3_joint: limit lower=-1.5708 upper=1.5708 effort=35.2 velocity=12.56 -> lower=-1.5708 upper=1.5708 effort=120 velocity=12.56
- joint leg_r4_joint: limit lower=0 upper=2.5307 effort=69.2 velocity=12.56 -> lower=0 upper=2.5307 effort=150 velocity=12.56
- joint leg_r5_joint: limit lower=-0.87266 upper=0.50614 effort=35.2 velocity=12.56 -> lower=-0.87266 upper=0.50614 effort=120 velocity=12.56
- joint leg_r6_joint: limit lower=-0.50614 upper=0.50614 effort=35.2 velocity=12.56 -> lower=-0.50614 upper=0.50614 effort=120 velocity=12.56

File: src/wbc_mjlab/CASBOT02_7dof/urdf/CASBOT02_ENCOS_23dof_shell_20251015.urdf (robot description, URDF)
Before this commit: robot CB02_URDF(ECS)130C, 32 links, 31 joints
Joints:
- joint leg_l1_joint: limit lower=-1.9199 upper=1.5708 effort=69.2 velocity=12.56 -> lower=-1.9199 upper=1.5708 effort=150 velocity=12.56
- joint leg_l2_joint: limit lower=-0.17453 upper=1.5708 effort=69.2 velocity=12.56 -> lower=-0.17453 upper=1.5708 effort=150 velocity=12.56
- joint leg_l3_joint: limit lower=-1.5708 upper=1.5708 effort=35.2 velocity=12.56 -> lower=-1.5708 upper=1.5708 effort=120 velocity=12.56
- joint leg_l4_joint: limit lower=0 upper=2.5307 effort=69.2 velocity=12.56 -> lower=0 upper=2.5307 effort=150 velocity=12.56
- joint leg_l5_joint: limit lower=-0.87266 upper=0.50614 effort=35.2 velocity=12.56 -> lower=-0.87266 upper=0.50614 effort=120 velocity=12.56
- joint leg_l6_joint: limit lower=-0.50614 upper=0.50614 effort=35.2 velocity=12.56 -> lower=-0.50614 upper=0.50614 effort=120 velocity=12.56
- joint leg_r1_joint: limit lower=-1.9199 upper=1.5708 effort=69.2 velocity=12.56 -> lower=-1.9199 upper=1.5708 effort=150 velocity=12.56
- joint leg_r2_joint: limit lower=-1.5708 upper=0.17453 effort=69.2 velocity=12.56 -> lower=-1.5708 upper=0.17453 effort=150 velocity=12.56
- joint leg_r3_joint: limit lower=-1.5708 upper=1.5708 effort=35.2 velocity=12.56 -> lower=-1.5708 upper=1.5708 effort=120 velocity=12.56
- joint leg_r4_joint: limit lower=0 upper=2.5307 effort=69.2 velocity=12.56 -> lower=0 upper=2.5307 effort=150 velocity=12.56
- joint leg_r5_joint: limit lower=-0.87266 upper=0.50614 effort=35.2 velocity=12.56 -> lower=-0.87266 upper=0.50614 effort=120 velocity=12.56
- joint leg_r6_joint: limit lower=-0.50614 upper=0.50614 effort=35.2 velocity=12.56 -> lower=-0.50614 upper=0.50614 effort=120 velocity=12.56

File: src/wbc_mjlab/CASBOT02_7dof/urdf/CASBOT02_ENCOS_7dof_shell_20251015.urdf (robot description, URDF)
Before this commit: robot CB02_URDF(ECS)130C, 32 links, 31 joints
Joints:
- joint leg_l1_joint: limit lower=-1.9199 upper=1.5708 effort=69.2 velocity=12.56 -> lower=-1.9199 upper=1.5708 effort=150 velocity=12.56
- joint leg_l2_joint: limit lower=-0.17453 upper=1.5708 effort=69.2 velocity=12.56 -> lower=-0.17453 upper=1.5708 effort=150 velocity=12.56
- joint leg_l3_joint: limit lower=-1.5708 upper=1.5708 effort=35.2 velocity=12.56 -> lower=-1.5708 upper=1.5708 effort=120 velocity=12.56
- joint leg_l4_joint: limit lower=0 upper=2.5307 effort=69.2 velocity=12.56 -> lower=0 upper=2.5307 effort=150 velocity=12.56
- joint leg_l5_joint: limit lower=-0.87266 upper=0.50614 effort=35.2 velocity=12.56 -> lower=-0.87266 upper=0.50614 effort=120 velocity=12.56
- joint leg_l6_joint: limit lower=-0.50614 upper=0.50614 effort=35.2 velocity=12.56 -> lower=-0.50614 upper=0.50614 effort=120 velocity=12.56
- joint leg_r1_joint: limit lower=-1.9199 upper=1.5708 effort=69.2 velocity=12.56 -> lower=-1.9199 upper=1.5708 effort=150 velocity=12.56
- joint leg_r2_joint: limit lower=-1.5708 upper=0.17453 effort=69.2 velocity=12.56 -> lower=-1.5708 upper=0.17453 effort=150 velocity=12.56
- joint leg_r3_joint: limit lower=-1.5708 upper=1.5708 effort=35.2 velocity=12.56 -> lower=-1.5708 upper=1.5708 effort=120 velocity=12.56
- joint leg_r4_joint: limit lower=0 upper=2.5307 effort=69.2 velocity=12.56 -> lower=0 upper=2.5307 effort=150 velocity=12.56
- joint leg_r5_joint: limit lower=-0.87266 upper=0.50614 effort=35.2 velocity=12.56 -> lower=-0.87266 upper=0.50614 effort=120 velocity=12.56
- joint leg_r6_joint: limit lower=-0.50614 upper=0.50614 effort=35.2 velocity=12.56 -> lower=-0.50614 upper=0.50614 effort=120 velocity=12.56

File: src/wbc_mjlab/CASBOT02_ENCOS_7dof_shell_20251015/Serial/urdf/CASBOT02_ENCOS_7dof_shell_20251015.urdf (robot description, URDF)
Before this commit: robot CB02_URDF(ECS)130C, 64 links, 63 joints
Joints:
- joint left_leg_ankle_pitch_joint: limit lower=-0.87266 upper=0.50614 effort=60 velocity=14 -> lower=-0.87266 upper=0.50614 effort=120 velocity=14
- joint left_leg_ankle_roll_joint: limit lower=-0.50614 upper=0.50614 effort=60 velocity=14 -> lower=-0.50614 upper=0.50614 effort=120 velocity=14
- joint left_leg_pelvic_yaw_joint: limit lower=-1.5708 upper=1.5708 effort=60 velocity=14 -> lower=-1.5708 upper=1.5708 effort=120 velocity=14
- joint right_leg_ankle_pitch_joint: limit lower=-0.87266 upper=0.50614 effort=60 velocity=14 -> lower=-0.87266 upper=0.50614 effort=120 velocity=14
- joint right_leg_ankle_roll_joint: limit lower=-0.50614 upper=0.50614 effort=60 velocity=14 -> lower=-0.50614 upper=0.50614 effort=120 velocity=14
- joint right_leg_pelvic_yaw_joint: limit lower=-1.5708 upper=1.5708 effort=60 velocity=14 -> lower=-1.5708 upper=1.5708 effort=120 velocity=14
